Commit message: Make RViz usable and the run repeatable
Both issues are usability/port problems, the algorithm is untouched.

RViz (config + display-only changes):
* /global_path asked for Transient Local while the publisher is Volatile, so the
  QoS was incompatible and the global path never rendered -> Volatile.
* there was no RobotModel display and jackal_tf.urdf had no geometry at all, so
  the robot was invisible -> URDF now carries the same body/wheel/lidar geometry
  as model.sdf, and the config adds a RobotModel display on /robot_description.
* /obs_predict_vis_pub publishes 25 predicted steps per obstacle (100+ cylinders
  per frame); draw every 5th step (kVisStride) so the prediction fan is legible.
  /obs_predict_pub, which the planner consumes, is unchanged.
* TF display off by default, smaller points, top-down orbit view, dark theme.

Repeat runs:
* gz-sim-main survives Ctrl+C and closing the Gazebo window only kills the GUI
  client, so the next launch died with 'Another world of the same name is
  running'. Add scripts/stop.sh (self-safe cleanup) and scripts/start.sh which
  cleans up before launching; run_experiment.sh uses it too.

Docs: run/stop instructions, what to look for in RViz, troubleshooting table,
and the final three-run results with the KF prediction-drift diagnosis.

File: src/mpc_dcbf_bringup/urdf/jackal_tf.urdf (robot description, URDF)
Before this commit: robot jackal_tf, 2 links, 1 joints
Links:
- added link front_left_wheel; visual cylinder length=0.04 radius=0.098
- added link front_right_wheel; visual cylinder length=0.04 radius=0.098
- added link rear_left_wheel; visual cylinder length=0.04 radius=0.098
- added link rear_right_wheel; visual cylinder length=0.04 radius=0.098
- link base_link: geometry visual box size=0.42 0.31 0.184
- link velodyne: geometry visual cylinder length=0.06 radius=0.05
Joints:
- added joint front_left_wheel_joint: type continuous, parent base_link, child front_left_wheel, origin xyz=0.131 0.187795 0.0345 rpy=0 0 0, axis 0 1 0
- added joint front_right_wheel_joint: type continuous, parent base_link, child front_right_wheel, origin xyz=0.131 -0.187795 0.0345 rpy=0 0 0, axis 0 1 0
- added joint rear_left_wheel_joint: type continuous, parent base_link, child rear_left_wheel, origin xyz=-0.131 0.187795 0.0345 rpy=0 0 0, axis 0 1 0
- added joint rear_right_wheel_joint: type continuous, parent base_link, child rear_right_wheel, origin xyz=-0.131 -0.187795 0.0345 rpy=0 0 0, axis 0 1 0
